File: kicad/keyboard.kicad_pcb (KiCad board)
At the start: 2 copper layers, 244 x 92 mm, 119 parts, among them SW1 SW_MX, SW10 SW_MX, SW11 SW_MX, SW12 SW_MX, SW13 SW_MX, SW14 SW_MX, SW15 SW_MX, SW16 SW_MX, SW17 SW_MX, SW18 SW_MX, SW19 SW_MX, SW2 SW_MX, SW20 SW_MX, SW21 SW_MX, SW22 SW_MX, SW23 SW_MX, SW24 SW_MX, SW25 SW_MX, SW26 SW_MX, SW27 SW_MX, SW28 SW_MX, SW29 SW_MX, SW3 SW_MX, SW30 SW_MX, SW31 SW_MX, SW32 SW_MX, SW33 SW_MX, SW34 SW_MX, SW35 SW_MX, SW36 SW_MX, SW37 SW_MX, SW38 SW_MX, SW39 SW_MX, SW4 SW_MX, SW40 SW_MX, SW41 SW_MX, SW42 SW_MX, SW43 SW_MX, SW44 SW_MX, SW45 SW_MX, SW46 SW_MX, SW47 SW_MX, SW48 SW_MX, SW49 SW_MX, SW5 SW_MX, SW50 SW_MX, SW51 SW_MX, SW52 SW_MX, SW53 SW_MX, SW54 SW_MX, SW55 SW_MX, SW56 SW_MX, SW57 SW_MX, SW58 SW_MX, SW59 SW_MX, SW6 SW_MX, SW7 SW_MX, SW8 SW_MX, SW9 SW_MX

Commit message: Update product name
Other:
- board text added: "Oxide © 2026 Jakub Świniarski"
- board text removed: "Oxide59 © 2026 Jakub Świniarski"
Changed lines of the file:
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@@
 		(layer "Edge.Cuts")
 	)
-	(gr_text "Oxide59\n\n© 2026 Jakub Świniarski"
+	(gr_text "Oxide\n\n© 2026 Jakub Świniarski"
 		(at 254.67 74.04 90)
 		(layer "B.SilkS")

Commit message: Update schematic and redesign PCB
Parts:
- added D60: D, Diode_THT:D_DO-35_SOD27_P7.62mm_Horizontal, B.Cu at (246.3, 59.1)
- added SW60: SW_MX, Button_Switch_Keyboard:SW_Cherry_MX_1.00u_PCB, F.Cu at (257.0, 51.5)
- A1: moved to B.Cu
- moved SW12 226.6 mm to (257.0, 127.5)
- moved D12 211.2 mm to (246.3, 137.7)
- moved SW47 209.3 mm to (238.0, 70.5)
- moved SW48 209.3 mm to (257.0, 70.5)
- moved D48 208.8 mm to (246.3, 80.7)
- moved D24 201.6 mm to (246.3, 116.1)
- moved SW23 201.5 mm to (238.0, 108.5)
- moved SW24 201.5 mm to (257.0, 108.5)
- moved D47 193.0 mm to (227.3, 80.7)
- moved D23 185.4 mm to (227.3, 118.7)
- moved SW36 183.0 mm to (257.0, 89.5)
- moved SW34 183.0 mm to (219.0, 89.5)
- moved SW35 183.0 mm to (238.0, 89.5)
- moved D35 182.9 mm to (227.3, 99.7)
- moved D36 182.9 mm to (246.3, 99.7)
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Connections:
- A1 pad 1: ROW4 -> unconnected-(A1-GPIO0-Pad1)
- A1 pad 11: COL6 -> COL7
- A1 pad 12: COL7 -> COL8
- A1 pad 14: COL8 -> COL9
- A1 pad 15: COL9 -> COL10
- A1 pad 16: COL10 -> COL11
- A1 pad 17: ROW2 -> unconnected-(A1-GPIO13-Pad17)
- A1 pad 19: unconnected-(A1-GPIO14-Pad19) -> ROW2
- A1 pad 2: COL0 -> COL2
- A1 pad 20: COL11 -> ROW0
- A1 pad 21: ROW0 -> ROW1
- A1 pad 22: ROW1 -> unconnected-(A1-GPIO17-Pad22)
- A1 pad 24: COL12 -> unconnected-(A1-GPIO18-Pad24)
- A1 pad 27: unconnected-(A1-GPIO21-Pad27) -> COL0
- A1 pad 29: unconnected-(A1-GPIO22-Pad29) -> COL1
- A1 pad 4: COL1 -> ROW4
- A1 pad 5: COL2 -> COL3
- A1 pad 6: COL3 -> COL6
- A1 pad 7: COL4 -> COL5
- A1 pad 9: COL5 -> COL4
- D1 pad 1: ROW4 -> ROW0
- D10 pad 1: ROW4 -> ROW0
- D11 pad 1: ROW4 -> ROW0
- D12 pad 1: ROW3 -> ROW0
- D13 pad 1: ROW3 -> ROW1
- D14 pad 1: ROW3 -> ROW1
- D15 pad 1: ROW3 -> ROW1
- D16 pad 1: ROW3 -> ROW1
- D17 pad 1: ROW3 -> ROW1
- D18 pad 1: ROW3 -> ROW1
- D19 pad 1: ROW3 -> ROW1
- D2 pad 1: ROW4 -> ROW0
- D20 pad 1: ROW3 -> ROW1
- D21 pad 1: ROW3 -> ROW1
- D22 pad 1: ROW3 -> ROW1
- D23 pad 1: ROW2 -> ROW1
- D24 pad 1: ROW2 -> ROW1
- D3 pad 1: ROW4 -> ROW0
- D34 pad 1: ROW1 -> ROW2
- D35 pad 1: ROW1 -> ROW2
- D36 pad 1: ROW1 -> ROW2
- D37 pad 1: ROW1 -> ROW3
- D38 pad 1: ROW1 -> ROW3
- D39 pad 1: ROW1 -> ROW3
- D4 pad 1: ROW4 -> ROW0
- D40 pad 1: ROW1 -> ROW3
- D41 pad 1: ROW1 -> ROW3
- D42 pad 1: ROW1 -> ROW3
- D43 pad 1: ROW1 -> ROW3
- D44 pad 1: ROW1 -> ROW3
- D45 pad 1: ROW1 -> ROW3
- D46 pad 1: ROW1 -> ROW3
- D47 pad 1: ROW0 -> ROW3
- D48 pad 1: ROW0 -> ROW3
- D49 pad 1: ROW0 -> ROW4
- D5 pad 1: ROW4 -> ROW0
- D50 pad 1: ROW0 -> ROW4
- D51 pad 1: ROW0 -> ROW4
- D52 pad 1: ROW0 -> ROW4
- D53 pad 1: ROW0 -> ROW4
- D54 pad 1: ROW0 -> ROW4
- D55 pad 1: ROW0 -> ROW4
- D56 pad 1: ROW0 -> ROW4
- D57 pad 1: ROW0 -> ROW4
- D58 pad 1: ROW0 -> ROW4
- D59 pad 1: ROW0 -> ROW4
- D6 pad 1: ROW4 -> ROW0
- D7 pad 1: ROW4 -> ROW0
- D8 pad 1: ROW4 -> ROW0
- D9 pad 1: ROW4 -> ROW0
- SW12 pad 1: COL0 -> COL11
- SW13 pad 1: COL1 -> COL0
- SW14 pad 1: COL2 -> COL1
- SW15 pad 1: COL3 -> COL2
- SW16 pad 1: COL4 -> COL3
- SW17 pad 1: COL5 -> COL4
- SW18 pad 1: COL6 -> COL5
- SW19 pad 1: COL7 -> COL6
- SW20 pad 1: COL8 -> COL7
- SW21 pad 1: COL9 -> COL8
- SW22 pad 1: COL10 -> COL9
- SW23 pad 1: COL0 -> COL10
- SW24 pad 1: COL1 -> COL11
- SW25 pad 1: COL2 -> COL0
- SW26 pad 1: COL3 -> COL1
- SW27 pad 1: COL4 -> COL2
- SW28 pad 1: COL5 -> COL3
- SW29 pad 1: COL6 -> COL4
- SW30 pad 1: COL7 -> COL5
- SW31 pad 1: COL8 -> COL6
- SW32 pad 1: COL9 -> COL7
- SW33 pad 1: COL10 -> COL8
- SW34 pad 1: COL0 -> COL9
- SW35 pad 1: COL1 -> COL10
- SW36 pad 1: COL2 -> COL11
- SW37 pad 1: COL3 -> COL0
- SW38 pad 1: COL4 -> COL1
- SW39 pad 1: COL5 -> COL2
- SW40 pad 1: COL6 -> COL3
- SW41 pad 1: COL7 -> COL4
- SW42 pad 1: COL8 -> COL5
- SW43 pad 1: COL9 -> COL6
- SW44 pad 1: COL10 -> COL7
- SW45 pad 1: COL11 -> COL8
- SW46 pad 1: COL12 -> COL9
- SW47 pad 1: COL0 -> COL10
- SW48 pad 1: COL1 -> COL11
- SW49 pad 1: COL2 -> COL0
- SW50 pad 1: COL3 -> COL1
- SW51 pad 1: COL4 -> COL2
- SW52 pad 1: COL5 -> COL3
- SW53 pad 1: COL6 -> COL4
- SW54 pad 1: COL7 -> COL5
- SW55 pad 1: COL8 -> COL6
- SW56 pad 1: COL9 -> COL7
- SW57 pad 1: COL10 -> COL8
- SW58 pad 1: COL11 -> COL9
- SW59 pad 1: COL12 -> COL10
Routing:
- net COL11: track 28.5 -> 241.4 mm
- net COL0: track 285.8 -> 105.1 mm, vias 1 -> 0
- net COL1: track 265.1 -> 86.9 mm, vias 1 -> 0
- net COL2: track 245.6 -> 82.9 mm, vias 1 -> 0
- net COL3: track 225.9 -> 88.7 mm, vias 1 -> 0
- net COL10: track 94.6 -> 222.6 mm
- net COL4: track 207.0 -> 109.2 mm, vias 1 -> 0
- net COL9: track 112.9 -> 204.2 mm
- net COL5: track 189.7 -> 128.7 mm, vias 1 -> 0
- net COL8: track 131.3 -> 186.9 mm
- net COL12: track 36.6 -> 0.00 mm
- net Net-(D51-A): track 5.30 -> 32.3 mm
- net Net-(D39-A): track 5.22 -> 31.9 mm
- net ROW0: track 263.2 -> 236.5 mm
- net Net-(D27-A): track 5.30 -> 32.0 mm
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Other:
- board size 244 x 92 mm -> 224.7 x 91.7 mm
- board text removed: "Oxide © 2026 Jakub Świniarski"

Commit message: Add copyright notice
Other:
- board text added: "© 2026 Jakub Świniarski"
